File: Calender.kicad_pcb (KiCad board)
At the start: 2 copper layers, 94 x 27.5 mm, 23 parts, among them J1 Screen, J2 USB_C_Receptacle_USB2.0_16P, J3 Power, SW1 RotaryEncoder_Switch, U1 ATSAMD21G18A-A, U3 MCP73871, U4 AMS1117-3.3, U5 ESP-WROOM-02

Commit message: all routing and stuff... definitely didn't forget to push
Parts:
- added C10: 100nF, Capacitor_SMD:C_0603_1608Metric, F.Cu at (185.0, 130.5)
- added C11: 100nF, Capacitor_SMD:C_0603_1608Metric, F.Cu at (174.5, 122.5)
- added C5: 1uF, Capacitor_SMD:C_0603_1608Metric, F.Cu at (176.5, 117.0)
- added C6: 100nF, Capacitor_SMD:C_0603_1608Metric, F.Cu at (193.0, 124.5)
- added C7: 100nF, Capacitor_SMD:C_0603_1608Metric, F.Cu at (194.0, 130.5)
- added C8: 100nF, Capacitor_SMD:C_0603_1608Metric, F.Cu at (193.0, 119.3)
- added C9: 100nF, Capacitor_SMD:C_0603_1608Metric, F.Cu at (189.0, 130.5)
- added R12: 10k, Resistor_SMD:R_0603_1608Metric, F.Cu at (231.2, 127.5)
- added R13: 10k, Resistor_SMD:R_0603_1608Metric, F.Cu at (169.0, 122.2)
- added SW2: SW_Push, Button_Switch_THT:SW_PUSH_6mm, F.Cu at (229.5, 117.5)
- added SW3: SW_Push, Button_Switch_THT:SW_PUSH_6mm, F.Cu at (214.0, 136.5)
- added SW4: SW_Push, Button_Switch_THT:SW_PUSH_6mm, F.Cu at (187.5, 136.5)
- J1: value Screen -> Conn_01x09; footprint Connector_PinHeader_2.54mm:PinHeader_1x09_P2.54mm_Vertical_SMD_Pin1Right -> Connector_PinHeader_1.00mm:PinHeader_1x09_P1.00mm_Vertical
- J3: footprint Connector_Phoenix_SPT:PhoenixContact_SPT_1.5_2-H-3.5_1x02_P3.5mm_Horizontal -> TerminalBlock:TerminalBlock_bornier-2_P5.08mm
- U4: moved to B.Cu
- moved C1 45.6 mm to (149.5, 133.5), turned to 180 degrees
- moved R1 44.9 mm to (152.5, 118.8), turned to -90 degrees
- moved R2 44.8 mm to (152.5, 123.2), turned to -90 degrees
- moved R6 42.8 mm to (159.0, 129.5)
- moved R5 41.7 mm to (159.5, 122.5), turned to 90 degrees
- moved R7 36.1 mm to (166.5, 116.5)
- moved R4 35.8 mm to (162.8, 119.0), turned to 180 degrees
- moved C2 34.4 mm to (159.0, 126.5), turned to 90 degrees
- moved R8 33.4 mm to (168.0, 127.5)
- moved R3 31.4 mm to (166.7, 119.0)
- moved C4 29.4 mm to (163.9, 127.5), turned to 180 degrees
- moved R11 26.4 mm to (231.0, 131.5)
- moved C3 21.1 mm to (172.3, 127.5)
- moved R10 14.3 mm to (217.0, 131.5)
- moved J3 10.2 mm to (146.7, 138.8), turned to 0 degrees
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Connections:
- J1 pad 1: (no net) -> OUT_3.3V
- J1 pad 2: (no net) -> GND
- J1 pad 3: (no net) -> DIN
- J1 pad 4: (no net) -> CLK
- J1 pad 5: (no net) -> CS
- J1 pad 6: (no net) -> DC
- J1 pad 7: (no net) -> RST
- J1 pad 8: (no net) -> BUSY
- J1 pad 9: (no net) -> OUT_3.3V
- U1 pad 10: unconnected-(U1-PA05-Pad10) -> TXD
- U1 pad 17: unconnected-(U1-VDDIO-Pad17) -> OUT_3.3V
- U1 pad 18: Net-(U1-GND-Pad18) -> GND
- U1 pad 25: unconnected-(U1-PA16-Pad25) -> PUSH_NEXT_DAY
- U1 pad 26: unconnected-(U1-PA17-Pad26) -> PUSH_BACK_DAY
- U1 pad 35: Net-(U1-GND-Pad18) -> GND
- U1 pad 36: unconnected-(U1-VDDIO-Pad36) -> OUT_3.3V
- U1 pad 42: Net-(U1-GND-Pad18) -> GND
- U1 pad 43: unconnected-(U1-VDDCORE-Pad43) -> Net-(U1-VDDCORE)
- U1 pad 44: unconnected-(U1-VDDIN-Pad44) -> OUT_3.3V
- U1 pad 5: unconnected-(U1-GNDANA-Pad5) -> Net-(U1-GNDANA)
- U1 pad 6: unconnected-(U1-VDDANA-Pad6) -> OUT_3.3V
- U1 pad 9: unconnected-(U1-PA04-Pad9) -> RXD
- U3 pad 6: unconnected-(U3-~{PG}-Pad6) -> Net-(U3-~{PG})
- U5 pad 8: unconnected-(U5-IO0-Pad8) -> OUT_3.3V
Routing:
- net GND: track 147.4 -> 258.3 mm, vias 2 -> 9
- net OUT_3.3V: track 57.8 -> 151.6 mm, vias 0 -> 8
- net BUSY: track 0.00 -> 66.9 mm, vias 0 -> 1
- net RST: track 0.00 -> 65.3 mm, vias 0 -> 1
- net vbus: track 91.3 -> 27.0 mm
- net DC: track 0.00 -> 63.5 mm, vias 0 -> 1
- net Net-(J2-CC1): track 64.0 -> 2.30 mm, vias 2 -> 0
- net DIN: track 0.00 -> 58.0 mm, vias 0 -> 1
- net CS: track 0.00 -> 55.3 mm, vias 0 -> 1
- net Net-(J2-CC2): track 56.9 -> 2.42 mm, vias 2 -> 0
- net CLK: track 0.00 -> 50.8 mm, vias 0 -> 1
- net RXD: track 0.00 -> 48.9 mm, vias 0 -> 2
- net Net-(U3-PROG1): track 51.4 -> 2.63 mm, vias 4 -> 0
- net TXD: track 0.00 -> 46.1 mm, vias 0 -> 2
- net Net-(U3-CE): track 59.9 -> 13.8 mm
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