File: Calender.kicad_pcb (KiCad board)
At the start: 2 copper layers, 94 x 27.5 mm, 35 parts, among them J1 Conn_01x09, J2 USB_C_Receptacle_USB2.0_16P, J3 Power, SW1 RotaryEncoder_Switch, SW2 SW_Push, SW3 SW_Push, SW4 SW_Push, U1 ATSAMD21G18A-A, U3 MCP73871, U4 AMS1117-3.3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

Commit message: PCB finished
Routing:
- net D-: track 53.6 -> 48.1 mm
- net D+: track 47.4 -> 45.8 mm, vias 5 -> 4
- net vbus: track 27.0 -> 27.7 mm
Changed lines of the file:
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@@
 	)
 	(segment
-		(start 149.595001 118.6)
-		(end 150.245 118.6)
+		(start 158.225 127.275)
+		(end 158 127.5)
 		(width 0.2)
 		(layer "F.Cu")
@@
 	)
 	(segment
-		(start 149.294 122.982824)
-		(end 149.294 118.901001)
+		(start 151.5 123.5)
+		(end 150.345 123.5)
 		(width 0.2)
 		(layer "F.Cu")
@@
 	)
 	(segment
-		(start 158.225 127.275)
-		(end 158 127.5)
+		(start 148.5 122.188824)
+		(end 148.5 119.695001)
 		(width 0.2)
 		(layer "F.Cu")
@@
 	)
 	(segment
-		(start 151.5 123.5)
-		(end 150.345 123.5)
+		(start 149.711176 123.4)
+		(end 148.5 122.188824)
 		(width 0.2)
 		(layer "F.Cu")
@@
 	)
 	(segment
+		(start 148.5 119.695001)
+		(end 149.595001 118.6)
+		(width 0.2)
+		(layer "F.Cu")
+		(net 23)
+	)
+	(segment
 		(start 159 127.275)
 		(end 158.225 127.275)
@@
 	)
 	(segment
-		(start 149.294 118.901001)
-		(end 149.595001 118.6)
+		(start 149.595001 118.6)
+		(end 150.245 118.6)
 		(width 0.2)
 		(layer "F.Cu")
@@
 	)
 	(segment
-		(start 149.711176 123.4)
-		(end 149.294 122.982824)
-		(width 0.2)
-		(layer "F.Cu")
-		(net 23)
-	)
-	(segment
 		(start 163.9375 124.9375)
 		(end 164.4375 124.9375)
@@
 	)
 	(segment
-		(start 167 123.5)
-		(end 166.650057 123.5)
-		(width 0.2)
-		(layer "B.Cu")
-		(net 26)
-	)
-	(segment
-		(start 165.399 125.399)
-		(end 165.899 125.899)
+		(start 177.15 118.85)
+		(end 177.15 119.975)
 		(width 0.2)
 		(layer "B.Cu")
@@
 	)
 	(segment
-		(start 169 126)
-		(end 169.182167 126)
+		(start 167 123.5)
+		(end 166.650057 123.5)
 		(width 0.2)
 		(layer "B.Cu")
@@
 	)
 	(segment
-		(start 169.182167 126)
-		(end 169.508524 126.326357)
+		(start 166.399 125.899)
+		(end 166.5 126)
 		(width 0.2)
 		(layer "B.Cu")
@@
 	)
 	(segment
-		(start 177.15 118.85)
-		(end 177.15 119.975)
+		(start 166.5 126)
+		(end 169.182167 126)
 		(width 0.2)
 		(layer "B.Cu")
@@
 	)
 	(segment
-		(start 165.899 125.899)
-		(end 166.399 125.899)
+		(start 169.182167 126)
+		(end 169.508524 126.326357)
 		(width 0.2)
 		(layer "B.Cu")
@@
 	)
 	(segment
-		(start 165.399 124.751057)
-		(end 165.399 125.399)
+		(start 236 122)
+		(end 229.5 122)
 		(width 0.2)
 		(layer "B.Cu")
@@
 	)
 	(segment
-		(start 166.650057 123.5)
-		(end 165.399 124.751057)
+		(start 204.5 141)
+		(end 214 141)
 		(width 0.2)
 		(layer "B.Cu")
@@
 	)
 	(segment
-		(start 166.5 126)
-		(end 169 126)
+		(start 165.399 125.399)
+		(end 165.899 125.899)
 		(width 0.2)
 		(layer "B.Cu")
@@
 	)
 	(segment
-		(start 236 122)
-		(end 229.5 122)
+		(start 214 141)
+		(end 220.5 141)
 		(width 0.2)
 		(layer "B.Cu")
@@
 	)
 	(segment
-		(start 204.5 141)
-		(end 214 141)
+		(start 165.399 124.751057)
+		(end 165.399 125.399)
 		(width 0.2)
 		(layer "B.Cu")
@@
 	)
 	(segment
-		(start 214 141)
-		(end 220.5 141)
+		(start 165.899 125.899)
+		(end 166.399 125.899)
 		(width 0.2)
 		(layer "B.Cu")
@@
 	)
 	(segment
-		(start 166.399 125.899)
-		(end 166.5 126)
+		(start 166.650057 123.5)
+		(end 165.399 124.751057)
 		(width 0.2)
 		(layer "B.Cu")
@@
 	)
 	(segment
+		(start 149.561176 121.25)
+		(end 150.245 121.25)
+		(width 0.2)
+		(layer "F.Cu")
+		(net 29)
+	)
+	(segment
 		(start 190.616535 120.640115)
 		(end 190.616535 120.616535)
@@
 	(segment
 		(start 150.245 120.25)
+		(end 149.561176 120.25)
+		(width 0.2)
+		(layer "F.Cu")
+		(net 29)
+	)
+	(segment
+		(start 150.245 120.25)
 		(end 151.75 120.25)
 		(width 0.2)
@@
 	)
 	(segment
-		(start 153.5 122)
-		(end 155 122)
+		(start 149.561176 120.25)
+		(end 149.294 120.517176)
 		(width 0.2)
 		(layer "F.Cu")
@@
 	)
 	(segment
-		(start 155 122)
-		(end 155 120)
+		(start 149.294 120.982824)
+		(end 149.561176 121.25)
 		(width 0.2)
 		(layer "F.Cu")
@@
 	)
 	(segment
-		(start 155 120)
+		(start 153.649 120.351)
 		(end 154 120)
 		(width 0.2)
@@
 	)
 	(segment
-		(start 152.75 121.25)
-		(end 153.5 122)
-		(width 0.2)
-		(layer "F.Cu")
-		(net 29)
-	)
-	(segment
-		(start 150.245 121.25)
-		(end 152.75 121.25)
-		(width 0.2)
-		(layer "F.Cu")
-		(net 29)
-	)
-	(segment
-		(start 153.649 120.351)
-		(end 154 120)
+		(start 149.294 120.517176)
+		(end 149.294 120.982824)
 		(width 0.2)
 		(layer "F.Cu")
@@
 	)
 	(segment
-		(start 151.25 121.75)
-		(end 150.245 121.75)
+		(start 151.196 121.017176)
+		(end 150.928824 120.75)
+		(width 0.2)
+		(layer "F.Cu")
+		(net 32)
+	)
+	(segment
+		(start 150.928824 120.75)
+		(end 150.245 120.75)
 		(width 0.2)
 		(layer "F.Cu")
@@
 	)
 	(segment
+		(start 150.928824 121.75)
+		(end 151.196 121.482824)
+		(width 0.2)
+		(layer "F.Cu")
+		(net 32)
+	)
+	(segment
+		(start 151.196 121.482824)
+		(end 151.196 121.017176)
+		(width 0.2)
+		(layer "F.Cu")
+		(net 32)
+	)
+	(segment
+		(start 150.245 121.75)
+		(end 150.928824 121.75)
+		(width 0.2)
+		(layer "F.Cu")
+		(net 32)
+	)
+	(segment
 		(start 150.245 120.75)
 		(end 150.247 120.752)
@@
 	)
 	(segment
-		(start 151.5 122)
-		(end 151.25 121.75)
-		(width 0.2)
-		(layer "F.Cu")
-		(net 32)
-	)
-	(segment
 		(start 187.5875 120.9125)
 		(end 189.4125 120.9125)
@@
 	)
 	(via
-		(at 151.5 122)
-		(size 0.6)
-		(drill 0.3)
-		(layers "F.Cu" "B.Cu")
-		(net 32)
-	)
-	(via
 		(at 154 121)
 		(size 0.6)
@@
 	)
 	(segment
-		(start 154 121)
-		(end 153 122)
-		(width 0.2)
-		(layer "B.Cu")
-		(net 32)
-	)
-	(segment
 		(start 173.5 117)
 		(end 174.101 116.399)
@@
 	)
 	(segment
-		(start 153 122)
-		(end 151.5 122)
-		(width 0.2)
-		(layer "B.Cu")
-		(net 32)
-	)
-	(segment
 		(start 174.101 116.399)
 		(end 182.899 116.399)
@@
 	)
 	(segment
-		(start 187.248943 127.899)
-		(end 187 127.899)
+		(start 189 129)
+		(end 188.298162 128.298162)
 		(width 0.2)
 		(layer "F.Cu")
@@
 	)
 	(segment
-		(start 187 127.899)
-		(end 187 126.325)
+		(start 187.648105 128.298162)
+		(end 187.248943 127.899)
 		(width 0.2)
 		(layer "F.Cu")
@@
 	)
 	(segment
-		(start 187.648105 128.298162)
-		(end 187.248943 127.899)
+		(start 187.248943 127.899)
+		(end 187 127.899)
 		(width 0.2)
 		(layer "F.Cu")
@@
 	)
 	(segment
-		(start 187.648105 129)
-		(end 187.648105 128.298162)
+		(start 187 127.899)
+		(end 187 126.325)
 		(width 0.2)
 		(layer "F.Cu")
@@
 	)
 	(segment
-		(start 189 129)
-		(end 187.648105 129)
+		(start 188.298162 128.298162)
+		(end 187.648105 128.298162)
 		(width 0.2)
 		(layer "F.Cu")
@@
 	)
 	(segment
-		(start 230.35 123.85)
-		(end 230.35 127.5)
+		(start 230.35 127.5)
+		(end 230.35 123.15)
 		(width 0.2)
 		(layer "F.Cu")
@@
 	)
 	(segment
-		(start 229.5 117.5)
-		(end 231.5 119.5)
-		(width 0.2)
-		(layer "F.Cu")
-		(net 68)
-	)
-	(segment
-		(start 231.5 122)
-		(end 230 123.5)
+		(start 231.5 119.5)
+		(end 231.5 122)
 		(width 0.2)
 		(layer "F.Cu")
@@
 	)
 	(segment
-		(start 231.5 119.5)
+		(start 230.35 123.15)
 		(end 231.5 122)
 		(width 0.2)
@@
 	)
 	(segment
-		(start 230 123.5)
-		(end 230.35 123.85)
+		(start 229.5 117.5)
+		(end 231.5 119.5)
 		(width 0.2)
 		(layer "F.Cu")

Commit message: Added prod files and bootloader stuff
Parts:
- added R14: 10k, Resistor_SMD:R_0603_1608Metric, B.Cu at (188.0, 116.0)
- moved C1 2.00 mm to (149.5, 131.5)
- moved J3 0.27 mm to (146.7, 138.5)
Connections:
- U1 pad 40: unconnected-(U1-~{RESET}-Pad40) -> RESET
- U1 pad 45: unconnected-(U1-PA30-Pad45) -> SWCLK
- U1 pad 46: unconnected-(U1-PA31-Pad46) -> SWDIO
Routing:
- net RESET: track 0.00 -> 11.8 mm, vias 0 -> 2
- net SWDIO: track 0.00 -> 6.24 mm, vias 0 -> 1
- net SWCLK: track 0.00 -> 5.60 mm, vias 0 -> 1
- net vbat: track 35.2 -> 38.8 mm
- net OUT_3.3V: track 151.6 -> 154.8 mm, vias 8 -> 10
- net D-: track 48.1 -> 50.7 mm
- net GND: track 258.3 -> 257.6 mm
Other:
- board text added: "RESET"
- board text added: "SWCLK"
- board text added: "SWDIO"

Commit message: The PCB should be good now for production
Parts:
- added G***: LOGO, LOGO, F.Cu at (203.2, 131.2)
- added R15: 1.5k, Resistor_SMD:R_0603_1608Metric, B.Cu at (187.5, 122.7)
- R14: moved to F.Cu
Connections:
- net Net-(U1-PB08) renamed ROT_A
- net Net-(U1-PB09) renamed ROT_B
Routing:
- net GND: track 257.6 -> 238.8 mm, vias 9 -> 53
- net D+: track 45.8 -> 51.5 mm, vias 4 -> 2
- net RESET: track 11.8 -> 6.54 mm, vias 2 -> 1
- net D-: track 50.7 -> 45.8 mm
- net OUT_3.3V: track 154.8 -> 159.2 mm, vias 10 -> 11
- net vbat: track 38.8 -> 39.9 mm
- net OUT_5V: track 16.1 -> 17.1 mm

Commit message: Fixed PCB changes/errors
Parts:
- added J4: Screen-2, Connector_PinHeader_2.54mm:PinHeader_1x04_P2.54mm_Vertical, F.Cu at (196.4, 124.0)
- R15, U4: moved to F.Cu
- moved R15 18.4 mm to (170.0, 117.0), turned to 180 degrees
- moved C11 5.65 mm to (173.2, 117.0), turned to 0 degrees
- moved R9 2.32 mm to (206.0, 116.8)
- moved G*** 0.35 mm to (203.0, 131.5)
- moved R13 0.28 mm to (168.7, 122.2)
Connections:
- U1 pad 27: unconnected-(U1-PA18-Pad27) -> SCK
- U1 pad 28: unconnected-(U1-PA19-Pad28) -> SDA
Routing:
- net SDA: track 0.00 -> 15.4 mm, vias 0 -> 1
- net SCK: track 0.00 -> 13.0 mm, vias 0 -> 1
- net GND: track 238.8 -> 232.5 mm, vias 53 -> 50
- net D+: track 51.5 -> 46.8 mm, vias 2 -> 3
- net OUT_5V: track 17.1 -> 21.3 mm, vias 2 -> 3
- net OUT_3.3V: track 159.2 -> 161.9 mm, vias 11 -> 8
- net Net-(U5-EN): track 5.26 -> 2.77 mm
- net Net-(U3-PROG3): track 19.8 -> 17.4 mm, vias 0 -> 2
- net Net-(U1-GNDANA): track 12.5 -> 10.6 mm, vias 2 -> 0
Other:
- board text added: "Designed by: ATY"

Commit message: Fixed more small PCB changed. Everything should be good now.
Parts:
- moved R5 0.84 mm to (160.3, 122.2)
Routing:
- net GND: track 232.5 -> 228.6 mm
- net Net-(U3-~{TE}): track 10.8 -> 8.17 mm
- net Net-(U3-PROG1): track 2.63 -> 1.73 mm

Commit message: have fun finishing the routing for it
Parts:
- added C12: 100nF, Capacitor_SMD:C_0603_1608Metric, F.Cu at (200.3, 147.3)
- added R16: 10kΩ, Resistor_SMD:R_0603_1608Metric, F.Cu at (200.3, 149.8)
- added R17: 10kΩ, Resistor_SMD:R_0603_1608Metric, F.Cu at (200.3, 152.3)
- added R18: 10kΩ, Resistor_SMD:R_0603_1608Metric, F.Cu at (200.3, 154.9)
- added R19: 10k, Resistor_SMD:R_0603_1608Metric, F.Cu at (206.8, 124.0)
- added TP1: TestPoint, TestPoint:TestPoint_Pad_4.0x4.0mm, B.Cu at (191.0, 147.6)
- added TP2: TestPoint, TestPoint:TestPoint_Pad_4.0x4.0mm, B.Cu at (191.0, 152.0)
- added TP3: TestPoint, TestPoint:TestPoint_Pad_4.0x4.0mm, B.Cu at (186.6, 147.6)
- added TP4: TestPoint, TestPoint:TestPoint_Pad_4.0x4.0mm, B.Cu at (186.6, 152.0)
- added TP5: TestPoint, TestPoint:TestPoint_Pad_4.0x4.0mm, B.Cu at (182.1, 147.6)
- added TP6: TestPoint, TestPoint:TestPoint_Pad_4.0x4.0mm, B.Cu at (182.1, 152.0)
- added TP7: TestPoint, TestPoint:TestPoint_Pad_4.0x4.0mm, B.Cu at (177.7, 147.6)
- added TP8: TestPoint, TestPoint:TestPoint_Pad_4.0x4.0mm, B.Cu at (177.7, 152.0)
- added U6: NAND, Package_SO:SOIC-8_5.3x5.3mm_P1.27mm, F.Cu at (209.0, 149.5)
Connections:
- U5 pad 6: unconnected-(U5-IO15-Pad6) -> Net-(U5-IO15)
Routing:
- net SWDIO: track 6.24 -> 0.00 mm, vias 1 -> 0
- net SWCLK: track 5.60 -> 0.00 mm, vias 1 -> 0
- net RESET: track 6.54 -> 2.28 mm, vias 1 -> 0
- net Net-(U5-IO15): track 0.00 -> 2.47 mm
- net GND: track 228.6 -> 230.1 mm

Commit message: Should be finished
Parts:
- moved TP8 57.1 mm to (225.0, 120.0)
- moved TP7 46.7 mm to (215.0, 119.5)
- moved TP1 40.0 mm to (220.0, 120.0)
- moved TP5 39.6 mm to (210.0, 119.5)
- moved TP4 36.0 mm to (202.0, 119.5)
- moved TP3 31.6 mm to (171.7, 119.7)
- moved TP6 26.9 mm to (158.0, 140.0)
- moved R17 16.6 mm to (199.6, 135.7)
- moved R18 16.4 mm to (197.0, 138.8), turned to 90 degrees
- moved TP2 15.8 mm to (182.0, 139.1)
- moved R16 14.4 mm to (208.5, 138.0), turned to 90 degrees
- moved C12 13.0 mm to (205.8, 135.5), turned to 180 degrees
- moved U6 11.9 mm to (202.5, 139.5)
Connections:
- R17 pad 2: CS_NAND MMCU -> CS_NAND
- U1 pad 12: unconnected-(U1-PA07-Pad12) -> CS_NAND
- U1 pad 15: unconnected-(U1-PA10-Pad15) -> MOSI
- U1 pad 16: unconnected-(U1-PA11-Pad16) -> MISO
- U6 pad 1: CS_NAND MMCU -> CS_NAND
- U6 pad 2: MISO TMCU -> MISO
- U6 pad 5: MOSI TMCU -> MOSI
- U6 pad 6: SCK TMCU -> SCK
Routing:
- net MOSI: track 0.00 -> 56.9 mm, vias 0 -> 2
- net MISO: track 0.00 -> 37.4 mm, vias 0 -> 2
- net SCK: track 13.0 -> 48.5 mm, vias 1 -> 3
- net SWCLK: track 0.00 -> 33.3 mm, vias 0 -> 1
- net D-: track 45.8 -> 78.4 mm, vias 2 -> 3
- net CS_NAND: track 0.00 -> 32.3 mm
- net SWDIO: track 0.00 -> 27.0 mm, vias 0 -> 3
- net +3.3V: track 0.00 -> 21.7 mm
- net RESET: track 2.28 -> 23.3 mm, vias 0 -> 1
- net D+: track 46.6 -> 67.3 mm, vias 3 -> 5
- net RXD: track 48.9 -> 65.5 mm, vias 2 -> 3
- net OUT_3.3V: track 161.6 -> 173.8 mm, vias 8 -> 9
- net TXD: track 46.1 -> 57.8 mm, vias 2 -> 4
- net Net-(U6-~{WP}/IO_{2}): track 0.00 -> 5.56 mm
- net GND: track 230.1 -> 234.7 mm, vias 50 -> 47
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Other:
- board text removed: "RESET"
- board text removed: "SWCLK"
- board text removed: "SWDIO"

Commit message: Added production files
Parts:
- removed TP6, TP7: TestPoint, TestPoint:TestPoint_Pad_4.0x4.0mm
Routing:
- net D-: track 78.4 -> 45.8 mm, vias 3 -> 2
- net GND: track 234.7 -> 204.5 mm, vias 47 -> 59
- net D+: track 67.3 -> 46.6 mm, vias 5 -> 3
- net SWDIO: track 27.0 -> 24.6 mm
- net MISO: track 37.4 -> 38.2 mm
- net SWCLK: track 33.3 -> 32.6 mm
- net vbat: track 39.9 -> 40.6 mm
- net CLK: track 51.2 -> 51.7 mm
- net vbus: track 27.7 -> 27.2 mm
