File: Calender.kicad_sch (KiCad schematic)
At the start: 35 parts, among them J1 Screen, J2 USB_C_Receptacle_USB2.0_16P, J3 Power, SW1 RotaryEncoder_Switch, SW2 SW_Push, SW3 SW_Push, SW4 SW_Push, U1 ATSAMD21G18A-A, U3 MCP73871, U4 AMS1117-3.3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

Commit message: all routing and stuff... definitely didn't forget to push
Parts:
- C10, C11, C5, C6, C7, C8, C9: footprint (none) -> Capacitor_SMD:C_0603_1608Metric
- J1: value Screen -> Conn_01x09; footprint Connector_PinHeader_2.54mm:PinHeader_1x09_P2.54mm_Vertical_SMD_Pin1Right -> Connector_PinHeader_1.00mm:PinHeader_1x09_P1.00mm_Vertical
- J3: footprint Connector_Phoenix_SPT:PhoenixContact_SPT_1.5_2-H-3.5_1x02_P3.5mm_Horizontal -> TerminalBlock:TerminalBlock_bornier-2_P5.08mm
- SW2, SW3, SW4: footprint (none) -> Button_Switch_THT:SW_PUSH_6mm
Connections:
- net BUSY: now also J1.8 (Pin_8); no longer J1.BUSY (IO25)
- net CLK: now also J1.4 (Pin_4); no longer J1.CLK (IO13)
- net CS: now also J1.5 (Pin_5); no longer J1.CS (IO15)
- net DC: now also J1.6 (Pin_6); no longer J1.DC (1O27)
- net DIN: now also J1.3 (Pin_3); no longer J1.DIN (IO14)
- net GND: now also J1.2 (Pin_2); no longer J1.GND (Pin_2)
- net OUT_3.3V: now also J1.1 (Pin_1), J1.9 (Pin_9); no longer J1.3.3V (VCC), J1.PWR (IO33)
- net RST: now also J1.7 (Pin_7); no longer J1.RST (IO26)
Changed lines of the file:
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@@
 			)
 		)
-		(property "Footprint" ""
+		(property "Footprint" "Capacitor_SMD:C_0603_1608Metric"
 			(at 53.34 26.3652 0)
 			(effects
@@
 			)
 		)
-		(property "Footprint" ""
+		(property "Footprint" "Capacitor_SMD:C_0603_1608Metric"
 			(at 71.12 18.0848 0)
 			(effects
@@
 			)
 		)
-		(property "Footprint" ""
+		(property "Footprint" "Capacitor_SMD:C_0603_1608Metric"
 			(at 64.4652 134.62 0)
 			(effects
@@
 			)
 		)
-		(property "Footprint" ""
+		(property "Footprint" "Capacitor_SMD:C_0603_1608Metric"
 			(at 71.12 23.1648 0)
 			(effects
@@
 			)
 		)
-		(property "Value" "Screen"
+		(property "Value" "Conn_01x09"
 			(at 133.35 48.2599 0)
 			(effects
@@
 			)
 		)
-		(property "Footprint" "Connector_PinHeader_2.54mm:PinHeader_1x09_P2.54mm_Vertical_SMD_Pin1Right"
+		(property "Footprint" "Connector_PinHeader_1.00mm:PinHeader_1x09_P1.00mm_Vertical"
 			(at 130.81 46.99 0)
 			(effects
@@
 			)
 		)
-		(pin "DIN"
+		(pin "7"
 		)
-		(pin "BUSY"
+		(pin "5"
 		)
-		(pin "3.3V"
+		(pin "2"
 		)
-		(pin "RST"
+		(pin "8"
 		)
-		(pin "CLK"
+		(pin "6"
 		)
-		(pin "DC"
+		(pin "9"
 		)
-		(pin "CS"
+		(pin "1"
 		)
-		(pin "PWR"
+		(pin "4"
 		)
-		(pin "GND"
+		(pin "3"
 		)
 		(instances
@@
 			)
 		)
-		(property "Footprint" ""
+		(property "Footprint" "Button_Switch_THT:SW_PUSH_6mm"
 			(at 266.7 135.89 0)
 			(effects
@@
 			)
 		)
-		(property "Footprint" ""
+		(property "Footprint" "Button_Switch_THT:SW_PUSH_6mm"
 			(at 92.71 114.3 0)
 			(effects
@@
 			)
 		)
-		(property "Footprint" "Connector_Phoenix_SPT:PhoenixContact_SPT_1.5_2-H-3.5_1x02_P3.5mm_Horizontal"
+		(property "Footprint" "TerminalBlock:TerminalBlock_bornier-2_P5.08mm"
 			(at 130.81 102.87 0)
 			(effects
@@
 			)
 		)
-		(property "Footprint" ""
+		(property "Footprint" "Capacitor_SMD:C_0603_1608Metric"
 			(at 45.72 31.4452 0)
 			(effects
@@
 			)
 		)
-		(property "Footprint" ""
+		(property "Footprint" "Capacitor_SMD:C_0603_1608Metric"
 			(at 55.88 17.4752 0)
 			(effects
@@
 			)
 		)
-		(property "Footprint" ""
+		(property "Footprint" "Button_Switch_THT:SW_PUSH_6mm"
 			(at 110.49 114.3 0)
 			(effects
@@
 			)
 		)
-		(property "Footprint" ""
+		(property "Footprint" "Capacitor_SMD:C_0603_1608Metric"
 			(at 55.88 22.5552 0)
 			(effects

Commit message: Added prod files and bootloader stuff
Parts:
- added R14: 10k, Resistor_SMD:R_0603_1608Metric, symbol Device:R
Connections:
- net OUT_3.3V: now also R14.1
- net RESET: now reaches U1.40 (~{RESET})
- net RESET: now also R14.2
- net SWCLK: now reaches U1.45 (PA30)
- net SWDIO: now reaches U1.46 (PA31)
Changed lines of the file:
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@@
+	)
+	(junction
+		(at 40.64 121.92)
+		(diameter 0)
+		(color 0 0 0 0)
 	)
 	(junction
@@
 	(wire
 		(pts
+			(xy 36.83 121.92) (xy 40.64 121.92)
+		)
+		(stroke
+			(width 0)
+			(type default)
+		)
+	)
+	(wire
+		(pts
 			(xy 193.04 73.66) (xy 195.58 73.66)
 		)
@@
 	(wire
 		(pts
+			(xy 36.83 114.3) (xy 43.18 114.3)
+		)
+		(stroke
+			(width 0)
+			(type default)
+		)
+	)
+	(wire
+		(pts
 			(xy 63.5 19.05) (xy 63.5 21.59)
 		)
@@
 		)
 	)
+	(wire
+		(pts
+			(xy 40.64 121.92) (xy 43.18 121.92)
+		)
+		(stroke
+			(width 0)
+			(type default)
+		)
+	)
 	(global_label "OUT_3.3V"
 		(shape input)
@@
 		)
 	)
+	(global_label "SWDIO"
+		(shape input)
+		(at 43.18 116.84 180)
+		(fields_autoplaced yes)
+		(effects
+			(font
+				(size 1.27 1.27)
+			)
+			(justify right)
+		)
+		(property "Intersheetrefs" "${INTERSHEET_REFS}"
+			(at 34.3286 116.84 0)
+			(effects
+				(font
+					(size 1.27 1.27)
+				)
+				(justify right)
+				(hide yes)
+			)
+		)
+	)
 	(global_label "OUT_5V"
 		(shape input)
@@
 		)
 	)
+	(global_label "SWCLK"
+		(shape input)
+		(at 36.83 114.3 180)
+		(fields_autoplaced yes)
+		(effects
+			(font
+				(size 1.27 1.27)
+			)
+			(justify right)
+		)
+		(property "Intersheetrefs" "${INTERSHEET_REFS}"
+			(at 27.6158 114.3 0)
+			(effects
+				(font
+					(size 1.27 1.27)
+				)
+				(justify right)
+				(hide yes)
+			)
+		)
+	)
 	(global_label "BUSY"
 		(shape input)
@@
 		)
 	)
+	(global_label "RESET"
+		(shape input)
+		(at 36.83 121.92 180)
+		(fields_autoplaced yes)
+		(effects
+			(font
+				(size 1.27 1.27)
+			)
+			(justify right)
+		)
+		(property "Intersheetrefs" "${INTERSHEET_REFS}"
+			(at 28.0997 121.92 0)
+			(effects
+				(font
+					(size 1.27 1.27)
+				)
+				(justify right)
+				(hide yes)
+			)
+		)
+	)
 	(global_label "OUT_3.3V"
 		(shape input)
@@
 		(property "Intersheetrefs" "${INTERSHEET_REFS}"
 			(at 25.0153 78.74 0)
+			(effects
+				(font
+					(size 1.27 1.27)
+				)
+				(justify right)
+				(hide yes)
+			)
+		)
+	)
+	(global_label "OUT_3.3V"
+		(shape input)
+		(at 40.64 129.54 270)
+		(fields_autoplaced yes)
+		(effects
+			(font
+				(size 1.27 1.27)
+			)
+			(justify right)
+		)
+		(property "Intersheetrefs" "${INTERSHEET_REFS}"
+			(at 40.64 141.2338 90)
 			(effects
 				(font
@@
 					(unit 1)
 				)
+			)
+		)
+	)
+	(symbol
+		(lib_id "Device:R")
+		(at 40.64 125.73 180)
+		(unit 1)
+		(exclude_from_sim no)
+		(in_bom yes)
+		(on_board yes)
+		(dnp no)
+		(property "Reference" "R14"
+			(at 43.18 125.73 90)
+			(effects
+				(font
+					(size 1.27 1.27)
+				)
+			)
+		)
+		(property "Value" "10k"
+			(at 40.64 125.73 90)
+			(effects
+				(font
+					(size 1.27 1.27)
+				)
+			)
+		)
+		(property "Footprint" "Resistor_SMD:R_0603_1608Metric"
+			(at 42.418 125.73 90)
+			(effects
+				(font
+					(size 1.27 1.27)
+				)
+				(hide yes)
+			)
+		)
+		(property "Datasheet" "~"
+			(at 40.64 125.73 0)
+			(effects
+				(font
+					(size 1.27 1.27)
+				)
+				(hide yes)
+			)
+		)
+		(property "Description" "Resistor"
+			(at 40.64 125.73 0)
+			(effects
+				(font
+					(size 1.27 1.27)
+				)
+				(hide yes)
+			)
+		)
+		(pin "2"
+		)
+		(pin "1"
+		)
+		(instances
+			(project "Calender"
+				(path "/7be0bee7-9169-4e67-9c75-05b4027453a4"
+					(reference "R14")
+					(unit 1)
+				)

Commit message: The PCB should be good now for production
Parts:
- added R15: 1.5k, Resistor_SMD:R_0603_1608Metric, symbol Device:R
Connections:
- net D+: now also R15.1
- net OUT_3.3V: now also R15.2
- net ROT_A: now reaches SW1.A, U1.7 (PB08)
- net ROT_B: now reaches SW1.B, U1.8 (PB09)
- no-connect marks 4 -> 32

Commit message: Fixed PCB changes/errors
Parts:
- added J4: Screen-2, Connector_PinHeader_2.54mm:PinHeader_1x04_P2.54mm_Vertical, symbol Connector:Conn_01x04_Pin
Connections:
- net GND: now also J4.1 (Pin_1)
- net OUT_3.3V: now also J4.2 (Pin_2)
- net SCK: now reaches U1.27 (PA18)
- net SCK: now also J4.3 (Pin_3)
- net SDA: now reaches U1.28 (PA19)
- net SDA: now also J4.4 (Pin_4)
- no-connect marks 32 -> 30

Commit message: have fun finishing the routing for it
Parts:
- added C12: 100nF, Capacitor_SMD:C_0603_1608Metric, symbol Device:C
- added R16, R17, R18: 10kΩ, Resistor_SMD:R_0603_1608Metric, symbol Device:R
- added R19: 10k, Resistor_SMD:R_0603_1608Metric, symbol Device:R
- added TP1, TP2, TP3, TP4, TP5, TP6, TP7, TP8: TestPoint, Connector_Pin:Pin_D1.0mm_L10.0mm_LooseFit, symbol Connector:TestPoint
- added U6: NAND, Package_SO:SOIC-8_5.3x5.3mm_P1.27mm, symbol Memory_Flash:W25Q128JVS
Connections:
- net D+: now also TP6.1
- net D-: now also TP7.1
- net GND: now also C12.2, R19.2, U6.4 (GND)
- net OUT_3.3V: now also TP8.1
- net RESET: now also TP3.1
- net RXD: now also TP2.1
- net SWCLK: now also TP5.1
- net SWDIO: now also TP4.1
- net TXD: now also TP1.1
- net at U5.6 (IO15): now also R19.1
- new net: R18.2, U6.3 (~{WP}/IO_{2})
- new net: R16.2, U6.7 (~{HOLD}/~{RESET}/IO_{3})
- new net +3.3V: C12.1, R16.1, R17.1, R18.1, U6.8 (VCC)
- new net CS_NAND MMCU: R17.2, U6.1 (~{CS})
- new net MISO TMCU: U6.2 (DO/IO_{1})
- new net MOSI TMCU: U6.5 (DI/IO_{0})
- new net SCK TMCU: U6.6 (CLK)
- no-connect marks 30 -> 29

Commit message: Should be finished
Connections:
- net CS_NAND MMCU is gone; now on net CS_NAND: R17.2, U6.1 (~{CS})
- net MISO TMCU is gone; now on net MISO: U6.2 (DO/IO_{1})
- net MOSI TMCU is gone; now on net MOSI: U6.5 (DI/IO_{0})
- net SCK TMCU is gone; now on net SCK: U6.6 (CLK)
- net CS_NAND: now reaches U1.12 (PA07)
- net MOSI: now reaches U1.15 (PA10)
- net MISO: now reaches U1.16 (PA11)
- no-connect marks 29 -> 26
Changed lines of the file:
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@@
-	)
-	(no_connect
-		(at 43.18 66.04)
 	)
 	(no_connect
@@
 	)
 	(no_connect
-		(at 43.18 63.5)
-	)
-	(no_connect
 		(at 257.81 133.35)
 	)
@@
 	)
 	(no_connect
-		(at 43.18 55.88)
-	)
-	(no_connect
 		(at 257.81 143.51)
 	)
@@
 		)
 	)
-	(global_label "CS_NAND MMCU"
+	(global_label "CS_NAND"
 		(shape input)
 		(at 101.6 160.02 180)
@@
 		)
 		(property "Intersheetrefs" "${INTERSHEET_REFS}"
-			(at 83.6772 160.02 0)
+			(at 90.1481 160.02 0)
 			(effects
 				(font
@@
 		)
 	)
+	(global_label "CS_NAND"
+		(shape input)
+		(at 43.18 55.88 180)
+		(fields_autoplaced yes)
+		(effects
+			(font
+				(size 1.27 1.27)
+			)
+			(justify right)
+		)
+		(property "Intersheetrefs" "${INTERSHEET_REFS}"
+			(at 31.7281 55.88 0)
+			(effects
+				(font
+					(size 1.27 1.27)
+				)
+				(justify right)
+				(hide yes)
+			)
+		)
+	)
 	(global_label "PUSH_1"
 		(shape input)
@@
 		)
 	)
-	(global_label "MOSI TMCU"
+	(global_label "MOSI"
 		(shape input)
 		(at 104.14 165.1 180)
@@
 		)
 		(property "Intersheetrefs" "${INTERSHEET_REFS}"
-			(at 90.5715 165.1 0)
+			(at 96.5586 165.1 0)
 			(effects
 				(font
@@
 		)
 	)
-	(global_label "MISO TMCU"
+	(global_label "MISO"
 		(shape input)
 		(at 104.14 167.64 180)
@@
 		)
 		(property "Intersheetrefs" "${INTERSHEET_REFS}"
-			(at 90.5715 167.64 0)
-			(effects
-				(font
-					(size 1.27 1.27)
-				)
-				(justify right)
-				(hide yes)
-			)
-		)
-	)
-	(global_label "SCK TMCU"
+			(at 96.5586 167.64 0)
+			(effects
+				(font
+					(size 1.27 1.27)
+				)
+				(justify right)
+				(hide yes)
+			)
+		)
+	)
+	(global_label "SCK"
 		(shape input)
 		(at 104.14 162.56 180)
@@
 		)
 		(property "Intersheetrefs" "${INTERSHEET_REFS}"
-			(at 91.4182 162.56 0)
+			(at 97.4053 162.56 0)
 			(effects
 				(font
@@
 		)
 	)
+	(global_label "MOSI"
+		(shape input)
+		(at 43.18 63.5 180)
+		(fields_autoplaced yes)
+		(effects
+			(font
+				(size 1.27 1.27)
+			)
+			(justify right)
+		)
+		(property "Intersheetrefs" "${INTERSHEET_REFS}"
+			(at 35.5986 63.5 0)
+			(effects
+				(font
+					(size 1.27 1.27)
+				)
+				(justify right)
+				(hide yes)
+			)
+		)
+	)
 	(global_label "CLK"
 		(shape input)
@@
 				(hide yes)
 			)
+		)
+	)
+	(global_label "MISO"
+		(shape input)
+		(at 43.18 66.04 180)
+		(fields_autoplaced yes)
+		(effects
+			(font
+				(size 1.27 1.27)
+			)
+			(justify right)
+		)
+		(property "Intersheetrefs" "${INTERSHEET_REFS}"
+			(at 35.5986 66.04 0)
+			(effects
+				(font
+					(size 1.27 1.27)
+				)
+				(justify right)
+				(hide yes)
+			)
